File: kicad/espboard.kicad_pcb (KiCad board)
At the start: 2 copper layers, 66 x 40.6 mm, 17 parts, among them J1 USB_OTG, P1 ftdi, P2 CONN_PWR, P3 CONN_IO, P4 usb_connector, U1 ESP-01v090, U2 LM1117-3.3

Commit message: Commit v2
Parts:
- moved REF*** 1.27 mm to (201.9, 97.8), turned to 90 degrees
Other:
- board text added: "3.3V"
- board text added: "5V"
- board text added: "GND"
- board text added: "IO0"
- board text added: "IO2"
- board text added: "NC"
- board text added: "RXD"
- board text added: "TXD"
Changed lines of the file:
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@@
-(kicad_pcb (version 4) (host pcbnew 4.0.6-e0-6349~53~ubuntu16.04.1)
+(kicad_pcb (version 4) (host pcbnew 4.0.7-e1-6374~58~ubuntu16.04.1)
   (general
     (links 41)
     (no_connects 0)
-    (area 144.679999 78.527 215.586191 119.645)
+    (area 144.679999 72.23 223.75 119.645)
     (thickness 1.6)
-    (drawings 11)
+    (drawings 24)
     (tracks 69)
     (zones 0)
@@
     (visible_elements FFFFFF7F)
     (pcbplotparams
-      (layerselection 0x000f0_80000001)
+      (layerselection 0x010f0_80000001)
       (usegerberextensions false)
       (excludeedgelayer true)
@@
   )
   (module Symbols:OSHW-Logo2_14.6x12mm_SilkScreen (layer F.Cu)
-    (at 200.66 97.79)
+    (at 201.93 97.79 90)
     (descr "Open Source Hardware Symbol")
     (tags "Logo Symbol OSHW")
     (attr virtual)
-    (fp_text reference REF*** (at 0 0) (layer F.SilkS) hide
-      (effects (font (size 1 1) (thickness 0.15)))
-    )
-    (fp_text value OSHW-Logo2_14.6x12mm_SilkScreen (at 0.75 0) (layer F.Fab) hide
+    (fp_text reference REF*** (at 0 0 90) (layer F.SilkS) hide
+      (effects (font (size 1 1) (thickness 0.15)))
+    )
+    (fp_text value OSHW-Logo2_14.6x12mm_SilkScreen (at 0.75 0 90) (layer F.Fab) hide
       (effects (font (size 1 1) (thickness 0.15)))
     )
@@
     (pad 1 thru_hole circle (at 0 0) (size 4.064 4.064) (drill 3.048) (layers *.Cu *.Mask))
   )
+  (gr_line (start 213.36 78.74) (end 213.36 119.38) (angle 90) (layer Edge.Cuts) (width 0.15))
+  (gr_line (start 147.32 119.38) (end 147.32 78.74) (angle 90) (layer Edge.Cuts) (width 0.15))
+  (dimension 40.64 (width 0.3) (layer Cmts.User)
+    (gr_text "40,640 mm" (at 218.52 99.06 90) (layer Cmts.User)
+      (effects (font (size 1.5 1.5) (thickness 0.3)))
+    )
+    (feature1 (pts (xy 213.36 78.74) (xy 219.87 78.74)))
+    (feature2 (pts (xy 213.36 119.38) (xy 219.87 119.38)))
+    (crossbar (pts (xy 217.17 119.38) (xy 217.17 78.74)))
+    (arrow1a (pts (xy 217.17 78.74) (xy 217.756421 79.866504)))
+    (arrow1b (pts (xy 217.17 78.74) (xy 216.583579 79.866504)))
+    (arrow2a (pts (xy 217.17 119.38) (xy 217.756421 118.253496)))
+    (arrow2b (pts (xy 217.17 119.38) (xy 216.583579 118.253496)))
+  )
+  (gr_text NC (at 190.5 111.76 90) (layer F.SilkS)
+    (effects (font (size 1.5 1.5) (thickness 0.3)) (justify right))
+  )
+  (gr_text NC (at 198.12 111.76 90) (layer F.SilkS)
+    (effects (font (size 1.5 1.5) (thickness 0.3)) (justify right))
+  )
+  (gr_text RXD (at 195.58 111.76 90) (layer F.SilkS)
+    (effects (font (size 1.5 1.5) (thickness 0.3)) (justify right))
+  )
+  (gr_text TXD (at 193.04 111.76 90) (layer F.SilkS)
+    (effects (font (size 1.5 1.5) (thickness 0.3)) (justify right))
+  )
+  (gr_text GND (at 185.42 111.76 90) (layer F.SilkS)
+    (effects (font (size 1.5 1.5) (thickness 0.3)) (justify right))
+  )
+  (gr_text RXD (at 203.2 83.82 90) (layer F.SilkS)
+    (effects (font (size 1.5 1.5) (thickness 0.3)) (justify left))
+  )
+  (gr_text TXD (at 200.66 83.82 90) (layer F.SilkS)
+    (effects (font (size 1.5 1.5) (thickness 0.3)) (justify left))
+  )
+  (gr_text IO0 (at 198.12 83.82 90) (layer F.SilkS)
+    (effects (font (size 1.5 1.5) (thickness 0.3)) (justify left))
+  )
+  (gr_text IO2 (at 195.58 83.82 90) (layer F.SilkS)
+    (effects (font (size 1.5 1.5) (thickness 0.3)) (justify left))
+  )
+  (gr_text 5V (at 185.42 83.82 90) (layer F.SilkS)
+    (effects (font (size 1.5 1.5) (thickness 0.3)) (justify left))
+  )
+  (gr_text 3.3V (at 187.96 83.82 90) (layer F.SilkS)
+    (effects (font (size 1.5 1.5) (thickness 0.3)) (justify left))
+  )
+  (gr_text GND (at 190.5 83.82 90) (layer F.SilkS)
+    (effects (font (size 1.5 1.5) (thickness 0.3)) (justify left))
+  )
+  (gr_text GND (at 193.04 83.82 90) (layer F.SilkS)
+    (effects (font (size 1.5 1.5) (thickness 0.3)) (justify left))
+  )
   (dimension 66.04 (width 0.3) (layer Cmts.User)
     (gr_text "66,040 mm" (at 180.34 73.58) (layer Cmts.User)
@@
     (arrow2b (pts (xy 147.32 74.93) (xy 148.446504 74.343579)))
   )
-  (dimension 40.64 (width 0.3) (layer Cmts.User)
-    (gr_text "40,640 mm" (at 218.52 99.06 90) (layer Cmts.User)
-      (effects (font (size 1.5 1.5) (thickness 0.3)))
-    )
-    (feature1 (pts (xy 213.36 78.74) (xy 219.87 78.74)))
-    (feature2 (pts (xy 213.36 119.38) (xy 219.87 119.38)))
-    (crossbar (pts (xy 217.17 119.38) (xy 217.17 78.74)))
-    (arrow1a (pts (xy 217.17 78.74) (xy 217.756421 79.866504)))
-    (arrow1b (pts (xy 217.17 78.74) (xy 216.583579 79.866504)))
-    (arrow2a (pts (xy 217.17 119.38) (xy 217.756421 118.253496)))
-    (arrow2b (pts (xy 217.17 119.38) (xy 216.583579 118.253496)))
-  )
-  (gr_line (start 147.32 119.38) (end 147.32 78.74) (angle 90) (layer Edge.Cuts) (width 0.15))
-  (gr_line (start 213.36 78.74) (end 213.36 119.38) (angle 90) (layer Edge.Cuts) (width 0.15))
   (gr_line (start 147.32 78.74) (end 213.36 78.74) (angle 90) (layer Edge.Cuts) (width 0.15))
   (gr_line (start 213.36 119.38) (end 147.32 119.38) (angle 90) (layer Edge.Cuts) (width 0.15))
